File: bloo.kicad_pcb (KiCad board)
At the start: 2 copper layers, 0 parts

Commit message: Removed green breakout board with generic 6 pin JST connector (3A)
Parts:
- added BT1: Battery_Cell, Connector_PinSocket_2.54mm:PinSocket_1x02_P2.54mm_Vertical, F.Cu at (85.5, 134.6)
- added BT_MH1: M2, MountingHole:MountingHole_2.2mm_M2, F.Cu at (67.6, 123.4)
- added BT_MH2: M2, MountingHole:MountingHole_2.2mm_M2, F.Cu at (67.6, 129.3)
- added BT_MH3: M2, MountingHole:MountingHole_2.2mm_M2, F.Cu at (73.6, 123.4)
- added BT_MH4: M2, MountingHole:MountingHole_2.2mm_M2, F.Cu at (73.6, 129.3)
- added C1: 0.1uF, Capacitor_SMD:C_1206_3216Metric_Pad1.33x1.80mm_HandSolder, F.Cu at (35.3, 112.0)
- added C10: 10uF(Tantalum), Capacitor_SMD:C_1206_3216Metric_Pad1.33x1.80mm_HandSolder, F.Cu at (35.3, 125.4)
- added C11: 10uF, Capacitor_SMD:C_1206_3216Metric_Pad1.33x1.80mm_HandSolder, F.Cu at (35.3, 128.7)
- added C12: 0.1uF, Capacitor_SMD:C_1206_3216Metric_Pad1.33x1.80mm_HandSolder, F.Cu at (41.4, 112.0)
- added C13: 0.1uF, Capacitor_SMD:C_1206_3216Metric_Pad1.33x1.80mm_HandSolder, F.Cu at (41.4, 115.3)
- added C14: 1uF, Capacitor_SMD:C_1206_3216Metric_Pad1.33x1.80mm_HandSolder, F.Cu at (41.4, 118.7)
- added C15: 1uF, Capacitor_SMD:C_1206_3216Metric_Pad1.33x1.80mm_HandSolder, F.Cu at (41.4, 122.0)
- added C16: 100uF, Capacitor_THT:CP_Radial_D6.3mm_P2.50mm, F.Cu at (58.1, 122.1)
- added C17: 1uF, Capacitor_SMD:C_1206_3216Metric_Pad1.33x1.80mm_HandSolder, F.Cu at (41.4, 125.4)
- added C18: 1uF, Capacitor_SMD:C_1206_3216Metric_Pad1.33x1.80mm_HandSolder, F.Cu at (41.4, 128.7)
- added C19: 0.1uF, Capacitor_SMD:C_1206_3216Metric_Pad1.33x1.80mm_HandSolder, F.Cu at (47.4, 112.0)
- added C2: 100uF, Capacitor_THT:CP_Radial_D6.3mm_P2.50mm, F.Cu at (58.1, 114.2)
- added C20: 1uF, Capacitor_SMD:C_1206_3216Metric_Pad1.33x1.80mm_HandSolder, F.Cu at (47.4, 115.3)
- added C21: 1uF, Capacitor_SMD:C_1206_3216Metric_Pad1.33x1.80mm_HandSolder, F.Cu at (47.4, 118.7)
- added C25: 10nF, Capacitor_SMD:C_1206_3216Metric_Pad1.33x1.80mm_HandSolder, F.Cu at (47.4, 122.0)
- added C3: 1uF, Capacitor_SMD:C_1206_3216Metric_Pad1.33x1.80mm_HandSolder, F.Cu at (35.3, 115.3)
- added C4: 0.1uF, Capacitor_SMD:C_1206_3216Metric_Pad1.33x1.80mm_HandSolder, F.Cu at (35.3, 118.7)
- added C9: 10uF, Capacitor_SMD:C_1206_3216Metric_Pad1.33x1.80mm_HandSolder, F.Cu at (35.3, 122.0)
- added D0: SFH4545, MM_Library:Emitter, F.Cu at (66.2, 110.6)
- added D1: SFH4545, MM_Library:Emitter, F.Cu at (71.8, 110.6)
- added D2: SFH4545, MM_Library:Emitter, F.Cu at (77.4, 110.6)
- added D3: SFH4545, MM_Library:Emitter, F.Cu at (82.9, 110.6)
- added D4: LED, LED_SMD:LED_0805_2012Metric_Pad1.15x1.40mm_HandSolder, F.Cu at (80.8, 133.8)
- added D5: LED, LED_SMD:LED_0805_2012Metric_Pad1.15x1.40mm_HandSolder, F.Cu at (80.8, 136.9)
- added D6: LED, LED_SMD:LED_0805_2012Metric_Pad1.15x1.40mm_HandSolder, F.Cu at (80.8, 139.9)
- added JP4: Jumper_2_Open, Jumper:SolderJumper-2_P1.3mm_Bridged_Pad1.0x1.5mm, F.Cu at (80.6, 143.2)
- added L1: 10uH, Inductor_SMD:L_1206_3216Metric_Pad1.42x1.75mm_HandSolder, F.Cu at (91.5, 56.5)
- added M1: M1_Conn_Alt, Connector_PinHeader_2.54mm:PinHeader_1x06_P2.54mm_Vertical, F.Cu at (95.9, 93.0)
- added M2: M2_Conn_Alt, Connector_PinHeader_2.54mm:PinHeader_1x06_P2.54mm_Vertical, F.Cu at (91.3, 93.0)
- added M_MH1: M2, MM_Library:Motor_mouse, F.Cu at (63.9, 68.7)
- added M_MH2: M2, MM_Library:Motor_mouse, F.Cu at (63.9, 96.4)
- added Q0: TEFT4300, MM_Library:Emitter, F.Cu at (88.5, 110.6)
- added Q1: TEFT4300, MM_Library:Emitter, F.Cu at (94.1, 110.6)
- added Q10: Q_NMOS_GSD, Package_TO_SOT_SMD:SOT-23, F.Cu at (52.8, 117.3)
- added Q11: Q_NMOS_GSD, Package_TO_SOT_SMD:SOT-23, F.Cu at (52.8, 122.0)
- added Q12: Q_NMOS_GSD, Package_TO_SOT_SMD:SOT-23, F.Cu at (52.8, 126.6)
- added Q2: TEFT4300, MM_Library:Emitter, F.Cu at (99.7, 110.6)
- added Q3: TEFT4300, MM_Library:Emitter, F.Cu at (105.3, 110.6)
- added Q9: Q_NMOS_GSD, Package_TO_SOT_SMD:SOT-23, F.Cu at (52.8, 112.7)
- added R1: 1.8k, Resistor_SMD:R_1206_3216Metric_Pad1.30x1.75mm_HandSolder, F.Cu at (91.5, 59.8)
- added R11: 47K, Resistor_SMD:R_1206_3216Metric_Pad1.30x1.75mm_HandSolder, F.Cu at (97.5, 63.1)
- added R12: 47K, Resistor_SMD:R_1206_3216Metric_Pad1.30x1.75mm_HandSolder, F.Cu at (97.5, 66.4)
- added R13: 47k, Resistor_SMD:R_1206_3216Metric_Pad1.30x1.75mm_HandSolder, F.Cu at (97.5, 69.7)
- added R14: 47k, Resistor_SMD:R_1206_3216Metric_Pad1.30x1.75mm_HandSolder, F.Cu at (97.5, 73.0)
- added R15: 47k, Resistor_SMD:R_1206_3216Metric_Pad1.30x1.75mm_HandSolder, F.Cu at (97.5, 76.3)
- added R16: 47k, Resistor_SMD:R_1206_3216Metric_Pad1.30x1.75mm_HandSolder, F.Cu at (97.5, 79.6)
- added R19: 750, Resistor_SMD:R_1206_3216Metric_Pad1.30x1.75mm_HandSolder, F.Cu at (103.4, 56.5)
- added R2: 1.8k, Resistor_SMD:R_1206_3216Metric_Pad1.30x1.75mm_HandSolder, F.Cu at (91.5, 63.1)
- added R20: 75, Resistor_SMD:R_1206_3216Metric_Pad1.30x1.75mm_HandSolder, F.Cu at (103.4, 59.8)
- added R21: 75, Resistor_SMD:R_1206_3216Metric_Pad1.30x1.75mm_HandSolder, F.Cu at (103.4, 63.1)
- added R22: 20K, Resistor_SMD:R_1206_3216Metric_Pad1.30x1.75mm_HandSolder, F.Cu at (103.4, 66.4)
- added R23: 10K, Resistor_SMD:R_1206_3216Metric_Pad1.30x1.75mm_HandSolder, F.Cu at (103.4, 69.7)
- added R24: 47K, Resistor_SMD:R_1206_3216Metric_Pad1.30x1.75mm_HandSolder, F.Cu at (103.4, 73.0)
- added R3: 1.8k, Resistor_SMD:R_1206_3216Metric_Pad1.30x1.75mm_HandSolder, F.Cu at (91.5, 66.4)
- added R4: 1.8k, Resistor_SMD:R_1206_3216Metric_Pad1.30x1.75mm_HandSolder, F.Cu at (91.5, 69.7)
- added R5: 35, Resistor_SMD:R_1206_3216Metric_Pad1.30x1.75mm_HandSolder, F.Cu at (91.5, 73.0)
- added R6: 35, Resistor_SMD:R_1206_3216Metric_Pad1.30x1.75mm_HandSolder, F.Cu at (91.5, 76.3)
- added R7: 35, Resistor_SMD:R_1206_3216Metric_Pad1.30x1.75mm_HandSolder, F.Cu at (91.5, 79.6)
- added R8: 35, Resistor_SMD:R_1206_3216Metric_Pad1.30x1.75mm_HandSolder, F.Cu at (97.5, 56.5)
- added R9: 47K, Resistor_SMD:R_1206_3216Metric_Pad1.30x1.75mm_HandSolder, F.Cu at (97.5, 59.8)
- added S1: EG1218, MM_Library:MM Switch, F.Cu at (57.2, 139.4)
- added SK1: M2, MountingHole:MountingHole_2.2mm_M2, F.Cu at (79.5, 123.4)
- added SK2: M2, MountingHole:MountingHole_2.2mm_M2, F.Cu at (79.5, 129.3)
- added SK3: M2, MountingHole:MountingHole_2.2mm_M2, F.Cu at (85.5, 123.4)
- added SK4: M2, MountingHole:MountingHole_2.2mm_M2, F.Cu at (85.5, 129.3)
- added SW1: SW, Button_Switch_SMD:SW_SPST_REED_CT05-XXXX-G1, F.Cu at (105.6, 122.9)
- added SW2: SW, Button_Switch_SMD:SW_SPST_REED_CT05-XXXX-G1, F.Cu at (105.6, 128.0)
- added SW3: SW, Button_Switch_SMD:SW_SPST_REED_CT05-XXXX-G1, F.Cu at (105.6, 133.0)
- added SW_RST1: SW, Button_Switch_SMD:SW_SPST_REED_CT05-XXXX-G1, F.Cu at (105.6, 138.1)
- added TP1: V_EXT_TP, Connector_PinHeader_2.54mm:PinHeader_1x01_P2.54mm_Vertical, F.Cu at (67.0, 134.6)
- added TP2: GND_TP, Connector_PinHeader_2.54mm:PinHeader_1x01_P2.54mm_Vertical, F.Cu at (67.0, 139.2)
- added TP3: TP_5V, Connector_PinHeader_2.54mm:PinHeader_1x01_P2.54mm_Vertical, F.Cu at (71.5, 134.6)
- added TP4: TP_3V3, Connector_PinHeader_2.54mm:PinHeader_1x01_P2.54mm_Vertical, F.Cu at (71.5, 139.2)
- added TP5: GND_TP, Connector_PinHeader_2.54mm:PinHeader_1x01_P2.54mm_Vertical, F.Cu at (76.1, 134.6)
- added TP6: GND_TP, Connector_PinHeader_2.54mm:PinHeader_1x01_P2.54mm_Vertical, F.Cu at (76.1, 139.2)
- added U1: YAAJ_BluePill_SWD_Breakout, MM_Library:STM32F103, F.Cu at (76.3, 80.5)
- added U2: L293D, Package_DIP:DIP-16_W7.62mm, F.Cu at (90.0, 122.5)
- added U3: LM1085-5.0, MM_Library:5V Voltage Reg, F.Cu at (41.2, 144.6)
- added U4: APE8865Y5-33-HF-3, Package_TO_SOT_SMD:SOT-23-5, F.Cu at (85.8, 141.9)
