File: _autosave-bloo.kicad_pcb (KiCad board)
At the start: 2 copper layers, 90 x 96 mm, 89 parts, among them J5 SWD_Header, M1 M1_Conn_Alt, M2 M2_Conn_Alt, Q0 TEFT4300, Q1 TEFT4300, Q10 Q_NMOS_GSD, Q11 Q_NMOS_GSD, Q12 Q_NMOS_GSD, Q2 TEFT4300, Q3 TEFT4300, Q9 Q_NMOS_GSD, SW1 SW, SW2 SW, SW3 SW, U1 YAAJ_BluePill_SWD_Breakout, U2 L293D, U3 LM1085-5.0, U4 APE8865Y5-33-HF-3, U5 BC832

Commit message: fixing DRC errors
Routing:
- net GND: track 0.00 -> 0.07 mm, vias 100 -> 101
Changed lines of the file:
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@@
 		(net 1)
 	)
+	(segment
+		(start 297.12 123.98)
+		(end 297.17 124.03)
+		(width 0.5)
+		(layer "F.Cu")
+		(net 2)
+	)
 	(via
 		(at 248.12 60.82)
@@
 	)
 	(via
+		(at 296.99 127.98)
+		(size 0.6)
+		(drill 0.3)
+		(layers "F.Cu" "B.Cu")
+		(free yes)
+		(net 2)
+	)
+	(via
 		(at 211.140994 76.548206)
 		(size 0.7)
@@
 	)
 	(via
-		(at 297.16 123.27)
-		(size 0.6)
-		(drill 0.3)
-		(layers "F.Cu" "B.Cu")
-		(free yes)
-		(net 2)
-	)
-	(via
-		(at 297.88 134.01)
-		(size 0.6)
-		(drill 0.3)
-		(layers "F.Cu" "B.Cu")
-		(free yes)
-		(net 2)
-	)
-	(via
 		(at 268.38 98.86)
 		(size 0.8)
@@
 	)
 	(via
+		(at 298.5 134.21)
+		(size 0.6)
+		(drill 0.3)
+		(layers "F.Cu" "B.Cu")
+		(free yes)
+		(net 2)
+	)
+	(via
 		(at 275.32 113.58)
 		(size 0.8)
@@
 	)
 	(via
+		(at 297.01 129)
+		(size 0.6)
+		(drill 0.3)
+		(layers "F.Cu" "B.Cu")
+		(free yes)
+		(net 2)
+	)
+	(via
 		(at 282.536857 100.107682)
 		(size 0.8)
@@
 	)
 	(via
+		(at 297.46 133.51)
+		(size 0.6)
+		(drill 0.3)
+		(layers "F.Cu" "B.Cu")
+		(free yes)
+		(net 2)
+	)
+	(via
 		(at 214.82 71.04)
 		(size 0.6)
@@
 	)
 	(via
-		(at 246.48 134.14)
-		(size 0.7)
-		(drill 0.4)
+		(at 297.12 123.09)
+		(size 0.6)
+		(drill 0.3)
 		(layers "F.Cu" "B.Cu")
 		(free yes)
@@
 	)
 	(via
-		(at 224.86 131.4)
+		(at 246.48 134.14)
 		(size 0.7)
 		(drill 0.4)
@@
 	)
 	(via
-		(at 293.42 123.83)
-		(size 0.6)
-		(drill 0.3)
+		(at 224.86 131.4)
+		(size 0.7)
+		(drill 0.4)
 		(layers "F.Cu" "B.Cu")
 		(free yes)
@@
 	)
 	(via
-		(at 297.14 133.36)
-		(size 0.6)
-		(drill 0.3)
-		(layers "F.Cu" "B.Cu")
-		(free yes)
-		(net 2)
-	)
-	(via
 		(at 253.39 127.61)
 		(size 0.8)
@@
 		(polygon
 			(pts
-				(xy 287.87 134.81) (xy 287.87 130.76) (xy 298.73 130.76) (xy 298.65 134.8) (xy 298.66 134.8)
+				(xy 287.81 134.44) (xy 287.87 130.76) (xy 296.51 130.84) (xy 296.41 134.32) (xy 296.4 134.43)
 			)
 		)
